File: kicad/GuitarMixer.kicad_sch (KiCad schematic)
At the start: 36 parts, among them J1 Conn_01x03_Pin, J2 Conn_01x03_Pin, J3 Conn_01x03_Pin, J4 Conn_01x02_Pin, J5 Conn_01x02_Pin, J6 Conn_01x03_Pin, Q1 2N5457, SW1 SW_SPST, U1 TL072, U2 TL072

Commit message: V1.0
Parts:
- added C10: 10pF, Capacitor_THT:C_Disc_D4.3mm_W1.9mm_P5.00mm, symbol Device:C_Small
- added C11: 100nF, Capacitor_THT:C_Rect_L7.2mm_W2.5mm_P5.00mm_FKS2_FKP2_MKS2_MKP2, symbol Device:C
- added R14: 10K, Resistor_THT:R_Axial_DIN0207_L6.3mm_D2.5mm_P10.16mm_Horizontal, symbol Device:R_Small
- C2: footprint Capacitor_THT:C_Disc_D4.7mm_W2.5mm_P5.00mm -> Capacitor_THT:C_Rect_L7.2mm_W2.5mm_P5.00mm_FKS2_FKP2_MKS2_MKP2
- C3: footprint Capacitor_THT:C_Rect_L7.0mm_W3.5mm_P5.00mm -> Capacitor_THT:C_Rect_L7.2mm_W2.5mm_P5.00mm_FKS2_FKP2_MKS2_MKP2
- C4: value 33nF -> 100nF; footprint Capacitor_THT:C_Disc_D4.7mm_W2.5mm_P5.00mm -> Capacitor_THT:C_Rect_L7.2mm_W2.5mm_P5.00mm_FKS2_FKP2_MKS2_MKP2
- C5, C6: value 100nF -> 1uF; footprint Capacitor_THT:C_Rect_L7.0mm_W3.5mm_P5.00mm -> Capacitor_THT:C_Rect_L7.2mm_W4.5mm_P5.00mm_FKS2_FKP2_MKS2_MKP2
- R10, R5, R7: value 100K -> 10K
Connections:
- net at R10.2, R12.2, U2.1: now also C10.2
- net at R10.1, R5.2, R7.2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: now also C10.1
- net +4V: now reaches C8.1, R8.1, R9.2, U2.3 (+), U2.5 (+)
- net at C6.1, U1.7: now also C11.2, R14.2; no longer U1.6 (-)
- new net: C11.1, R14.1, U1.6 (-)
Other:
- note added: "Notes: 1. Ensure that the input jacks used switch the tip pins to GND when nothing plugged in"
- note removed: "Notes: 1. A bias trimmer between R8 and R9 may help reduce distortion on U2 (or just tie to earth?) 2. Ensure that the input jacks used switch the tip pins to GND when nothing plugged in 3. U1B might benefit from a resistor and capacitor in the negative feedback loop so there is some amplification"
- title: GuitarMixer -> AEGM - Acoustic Electric Guitar Mixer
- moved on the sheet: C3, C5, C6, C7, C8, C9, D1, J2, J3, J4, J5, J6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

Commit message: Redid the feedback on the non-inverting amplifier for electric guitar
Parts:
- added R15: 1K, Resistor_THT:R_Axial_DIN0207_L6.3mm_D2.5mm_P10.16mm_Horizontal, symbol Device:R_Small
- R14: value 10K -> 1K
Connections:
- net Earth: now also R15.2
- net at C11.1, R14.1, U1.6 (-): now also R15.1
Changed lines of the file:
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@@
 	(title_block
 		(title "AEGM - Acoustic Electric Guitar Mixer")
-		(date "2025-10-09")
-		(rev "V1.0")
+		(date "2025-10-17")
+		(rev "V1.1")
 		(company "Andrew Martin")
 		(comment 1 "Fully working")
+		(comment 2 "V1.1 Redid feedback on the non-inverting amp for electric")
 	)
 	(text "Notes:\n1. Ensure that the input jacks used switch the tip pins to GND when nothing plugged in\n\n\n"
@@
 	)
 	(junction
+		(at 91.44 102.87)
+		(diameter 0)
+		(color 0 0 0 0)
+	)
+	(junction
 		(at 46.99 140.97)
 		(diameter 0)
@@
 	(wire
 		(pts
+			(xy 91.44 91.44) (xy 100.33 91.44)
+		)
+		(stroke
+			(width 0)
+			(type default)
+		)
+	)
+	(wire
+		(pts
 			(xy 125.73 77.47) (xy 128.27 77.47)
 		)
@@
 	(wire
 		(pts
-			(xy 62.23 102.87) (xy 128.27 102.87)
+			(xy 62.23 102.87) (xy 91.44 102.87)
 		)
 		(stroke
@@
 	(wire
 		(pts
+			(xy 91.44 99.06) (xy 91.44 102.87)
+		)
+		(stroke
+			(width 0)
+			(type default)
+		)
+	)
+	(wire
+		(pts
 			(xy 55.88 60.96) (xy 62.23 60.96)
 		)
@@
 	(wire
 		(pts
+			(xy 91.44 102.87) (xy 128.27 102.87)
+		)
+		(stroke
+			(width 0)
+			(type default)
+		)
+	)
+	(wire
+		(pts
 			(xy 45.72 39.37) (xy 50.8 39.37)
 		)
@@
 	(wire
 		(pts
+			(xy 91.44 93.98) (xy 91.44 91.44)
+		)
+		(stroke
+			(width 0)
+			(type default)
+		)
+	)
+	(wire
+		(pts
 			(xy 45.72 55.88) (xy 45.72 60.96)
 		)
@@
 			)
 		)
-		(property "Value" "10K"
+		(property "Value" "1K"
 			(at 109.22 88.9 90)
 			(effects
@@
 					(unit 1)
 				)
+			)
+		)
+	)
+	(symbol
+		(lib_id "Device:R_Small")
+		(at 91.44 96.52 0)
+		(unit 1)
+		(exclude_from_sim no)
+		(in_bom yes)
+		(on_board yes)
+		(dnp no)
+		(fields_autoplaced yes)
+		(property "Reference" "R15"
+			(at 93.98 95.2499 0)
+			(effects
+				(font
+					(size 1.27 1.27)
+				)
+				(justify left)
+			)
+		)
+		(property "Value" "1K"
+			(at 93.98 97.7899 0)
+			(effects
+				(font
+					(size 1.27 1.27)
+				)
+				(justify left)
+			)
+		)
+		(property "Footprint" "Resistor_THT:R_Axial_DIN0207_L6.3mm_D2.5mm_P10.16mm_Horizontal"
+			(at 91.44 96.52 0)
+			(effects
+				(font
+					(size 1.27 1.27)
+				)
+				(hide yes)
+			)
+		)
+		(property "Datasheet" "~"
+			(at 91.44 96.52 0)
+			(effects
+				(font
+					(size 1.27 1.27)
+				)
+				(hide yes)
+			)
+		)
+		(property "Description" "Resistor, small symbol"
+			(at 91.44 96.52 0)
+			(effects
+				(font
+					(size 1.27 1.27)
+				)
+				(hide yes)
+			)
+		)
+		(pin "2"
+		)
+		(pin "1"
+		)
+		(instances
+			(project ""
+				(path "/dd0f4f85-8a06-4c68-92dc-fefacd0af10a"
+					(reference "R15")
+					(unit 1)
+				)
