File: kicad/GuitarMixer.kicad_pcb (KiCad board)
At the start: 2 copper layers, 83.7 x 45.6 mm, 46 parts, among them J1 Conn_01x03_Pin, J2 Conn_01x03_Pin, J3 Conn_01x03_Pin, J4 Conn_01x02_Pin, J5 Conn_01x02_Pin, J6 Conn_01x03_Pin, Q1 2N5457, SW1 SW_SPST, U1 TL072, U2 TL072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

Commit message: Moved the voltage setting resistors and created gerber and distribution files
Parts:
- D1: footprint Diode_THT:D_DO-35_SOD27_P2.54mm_Vertical_AnodeUp -> Diode_THT:D_DO-35_SOD27_P7.62mm_Horizontal
- moved R5 118.9 mm to (150.3, 112.9), turned to 0 degrees
- moved R6 108.4 mm to (144.7, 112.9), turned to 0 degrees
- moved D1 86.8 mm to (161.6, 113.2), turned to 90 degrees
- moved C1 83.2 mm to (154.8, 88.9)
- moved C102 83.2 mm to (109.8, 80.8)
- moved C105 83.2 mm to (150.3, 79.2)
- moved C205 83.2 mm to (165.8, 79.5)
- moved C8 83.2 mm to (144.9, 98.5)
- moved C9 83.2 mm to (169.6, 84.1)
- moved J2 83.2 mm to (140.2, 76.3)
- moved J3 83.2 mm to (155.7, 76.3)
- moved J5 83.2 mm to (172.5, 76.3)
- moved R1 83.2 mm to (159.7, 93.0)
- moved R1011 83.2 mm to (126.8, 73.8)
- moved R1012 83.2 mm to (126.8, 87.6)
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Routing:
- net Net-(U3-ADJ): track 46.0 -> 10.5 mm
- net +9VA: track 115.3 -> 122.8 mm
- net Earth: track 319.3 -> 326.0 mm
- net +4.5V: track 155.7 -> 158.2 mm
- net Net-(D1-A): track 4.57 -> 6.35 mm
Other:
- board text added: "TP+"
- board text added: "TP-"
